File: lpc812-nrf24l01-8ch-receiver/electronics/lpc812-nrf24l01-8ch-receiver.sch (KiCad schematic (older format))
At the start: 24 parts, among them J1 CH1, J2 CH2, J3 CH3/Rx, J4 CH4/Tx, J5 CH5, J6 CH6, J7 CH7, J8 CH8, SW1 BIND/ISP, U1 MCP1703A-3302_SOT23, U2 LPC812M101JDH20, U3 NRF24L01_Breakout, Y1 16MHz

Commit message: Work on initial layout
Parts:
- U3: footprint RF_Module:nRF24L01_Breakout -> nordic-semiconductor:nrf24l01-E01-ML01IPX
Connections:
- net labels added: CH1-Rx, CH3, CH4, CH6-Tx
- net labels removed: CH1, CH3-Rx, CH4-Tx, CH6
Other:
- note added: "The following MCU pins can not be moved:\nCH3-Rx PIO0: ISP UART Rx (you can assign another RC channel though!)\nCH4-Tx PIO4: ISP UART Tx (you can assign another RC channel though!)\nBIND-ISP PIO12: ISP entry button\nXTALIN PIO8: crystal\nXTALIN PIO9: crystal"
Changed lines of the file:
@@
 F 0 "U3" H 7028 1978 50  0000 L CNN
 F 1 "NRF24L01_Breakout" H 7028 1887 50  0000 L CNN
-F 2 "RF_Module:nRF24L01_Breakout" H 6700 2600 50  0001 L CIN
+F 2 "nordic-semiconductor:nrf24l01-E01-ML01IPX" H 6700 2600 50  0001 L CIN
 F 3 "http://www.nordicsemi.com/eng/content/download/2730/34105/file/nRF24L01_Product_Specification_v2_0.pdf" H 6550 1900 50  0001 C CNN
 	1    6550 2000
@@
 L Device:R_Pack04 RN1
 U 1 1 5B9B56F7
-P 9000 1700
-F 0 "RN1" V 8583 1700 50  0000 C CNN
-F 1 "R_Pack04" V 8674 1700 50  0000 C CNN
-F 2 "Resistor_SMD:R_Array_Concave_4x0603" V 9275 1700 50  0001 C CNN
-F 3 "~" H 9000 1700 50  0001 C CNN
-	1    9000 1700
-	0    1    1    0
+P 9000 1600
+F 0 "RN1" V 8583 1600 50  0000 C CNN
+F 1 "R_Pack04" V 8674 1600 50  0000 C CNN
+F 2 "Resistor_SMD:R_Array_Concave_4x0603" V 9275 1600 50  0001 C CNN
+F 3 "~" H 9000 1600 50  0001 C CNN
+	1    9000 1600
+	0    1    -1   0
 $EndComp
 $Comp
 L Device:R_Pack04 RN2
 U 1 1 5B9B57C3
-P 9000 3700
-F 0 "RN2" V 8583 3700 50  0000 C CNN
-F 1 "R_Pack04" V 8674 3700 50  0000 C CNN
-F 2 "Resistor_SMD:R_Array_Concave_4x0603" V 9275 3700 50  0001 C CNN
-F 3 "~" H 9000 3700 50  0001 C CNN
-	1    9000 3700
-	0    1    1    0
+P 9000 3600
+F 0 "RN2" V 8583 3600 50  0000 C CNN
+F 1 "R_Pack04" V 8674 3600 50  0000 C CNN
+F 2 "Resistor_SMD:R_Array_Concave_4x0603" V 9275 3600 50  0001 C CNN
+F 3 "~" H 9000 3600 50  0001 C CNN
+	1    9000 3600
+	0    1    -1   0
 $EndComp
 $Comp
@@
 	6100 6250 6100 6400
 Text Label 5100 6250 0    50   ~ 0
+XTALOUT
+Text Label 6100 6250 2    50   ~ 0
 XTALIN
-Text Label 6100 6250 2    50   ~ 0
-XTALOUT
 Wire Wire Line
 	1300 6150 1300 6250
@@
 	2500 2700 1900 2700
 Text Label 1900 2700 0    50   ~ 0
-CH3-Rx
+CH1-Rx
 Wire Wire Line
 	2500 2800 1900 2800
@@
 	2500 3400 1900 3400
 Text Label 1900 2800 0    50   ~ 0
-SCK
+CH5
 Text Label 1900 2900 0    50   ~ 0
 MOSI
 Text Label 1900 3000 0    50   ~ 0
-CSN
+MISO
 Text Label 1900 3100 0    50   ~ 0
-CH4-Tx
+CH6-Tx
 Text Label 1900 3200 0    50   ~ 0
-LED
+IRQ
 Text Label 1900 3300 0    50   ~ 0
-CH1
+CH3
 Text Label 1900 3400 0    50   ~ 0
-CH2
+CH4
 Wire Wire Line
 	3900 2800 4600 2800
 Text Label 4600 2800 2    50   ~ 0
-IRQ
+CSN
 Wire Wire Line
 	3900 2900 4600 2900
@@
 	3900 3000 4600 3000
 Text Label 4600 2900 2    50   ~ 0
-MISO
+SCK
 Text Label 4600 3000 2    50   ~ 0
 BIND-ISP
@@
 	3900 3200 4600 3200
 Text Label 4600 3100 2    50   ~ 0
-CE
+CH8
 Text Label 4600 3300 2    50   ~ 0
-CH6
+LED
 Wire Wire Line
 	3900 3300 4600 3300
 Text Label 4600 3400 2    50   ~ 0
-CH7
+CE
 Wire Wire Line
 	3900 3400 4600 3400
 Text Label 4600 3500 2    50   ~ 0
-CH8
+CH7
 $Comp
 L power:GND #PWR0117
@@
 	8050 3800 8800 3800
 Text Label 8050 1500 0    50   ~ 0
-CH1
+CH1-Rx
 Text Label 8050 1600 0    50   ~ 0
 CH2
 Text Label 8050 1700 0    50   ~ 0
-CH3-Rx
+CH3
 Text Label 8050 1800 0    50   ~ 0
-CH4-Tx
+CH4
 Text Label 8050 3500 0    50   ~ 0
 CH5
 Text Label 8050 3600 0    50   ~ 0
-CH6
+CH6-Tx
 Text Label 8050 3700 0    50   ~ 0
 CH7
@@
 	3900 3500 4600 3500
 Text Label 4600 3200 2    50   ~ 0
-CH5
+CH2
 $Comp
 L power:PWR_FLAG #FLG0102
@@
 Wire Wire Line
 	10000 6100 10000 6200
+Text Notes 1750 4950 0    50   ~ 0
+The following MCU pins can not be moved:\nCH3-Rx PIO0: ISP UART Rx (you can assign another RC channel though!)\nCH4-Tx PIO4: ISP UART Tx (you can assign another RC channel though!)\nBIND-ISP PIO12: ISP entry button\nXTALIN PIO8: crystal\nXTALIN PIO9: crystal
 $EndSCHEMATC

Commit message: Add correct symbol for nRF24 module
Parts:
- removed C2: 1u/16V, Capacitor_SMD:C_0805_2012Metric_Pad1.15x1.40mm_HandSolder, symbol Device:C
- removed U3: NRF24L01_Breakout, nordic-semiconductor:nrf24l01-E01-ML01IPX, symbol RF:NRF24L01_Breakout
- added U3: NRF24L01_E01_ML01, nordic-semiconductor:nrf24l01-E01-ML01IPX, symbol nrf24l01_E01-ML01:NRF24L01_E01_ML01
- C3, C5: value CP -> 47u/6.3V
Connections:
- wire segments 122 -> 119
Changed lines of the file:
@@
 EESchema Schematic File Version 4
+LIBS:lpc812-nrf24l01-8ch-receiver-cache
 EELAYER 26 0
 EELAYER END
@@
 $EndComp
 $Comp
-L RF:NRF24L01_Breakout U3
-U 1 1 5B9B4FAE
-P 6550 2000
-F 0 "U3" H 7028 1978 50  0000 L CNN
-F 1 "NRF24L01_Breakout" H 7028 1887 50  0000 L CNN
-F 2 "nordic-semiconductor:nrf24l01-E01-ML01IPX" H 6700 2600 50  0001 L CIN
-F 3 "http://www.nordicsemi.com/eng/content/download/2730/34105/file/nRF24L01_Product_Specification_v2_0.pdf" H 6550 1900 50  0001 C CNN
-	1    6550 2000
-	1    0    0    -1
-$EndComp
-$Comp
 L Regulator_Linear:MCP1703A-3302_SOT23 U1
 U 1 1 5B9B50CE
@@
 $EndComp
 $Comp
-L Device:C C2
-U 1 1 5B9B52DA
-P 2450 6500
-F 0 "C2" H 2565 6546 50  0000 L CNN
-F 1 "1u/16V" H 2565 6455 50  0000 L CNN
-F 2 "Capacitor_SMD:C_0805_2012Metric_Pad1.15x1.40mm_HandSolder" H 2488 6350 50  0001 C CNN
-F 3 "~" H 2450 6500 50  0001 C CNN
-	1    2450 6500
-	1    0    0    -1
-$EndComp
-$Comp
 L Device:CP C3
 U 1 1 5B9B535A
-P 3200 6500
-F 0 "C3" H 3318 6546 50  0000 L CNN
-F 1 "CP" H 3318 6455 50  0000 L CNN
-F 2 "Capacitor_SMD:C_0805_2012Metric_Pad1.15x1.40mm_HandSolder" H 3238 6350 50  0001 C CNN
-F 3 "~" H 3200 6500 50  0001 C CNN
-	1    3200 6500
+P 2650 6500
+F 0 "C3" H 2768 6546 50  0000 L CNN
+F 1 "47u/6.3V" H 2650 6400 50  0000 L CNN
+F 2 "Capacitor_SMD:C_0805_2012Metric_Pad1.15x1.40mm_HandSolder" H 2688 6350 50  0001 C CNN
+F 3 "~" H 2650 6500 50  0001 C CNN
+	1    2650 6500
 	1    0    0    -1
 $EndComp
@@
 L power:VCC #PWR0101
 U 1 1 5B9B64E9
-P 3650 6100
-F 0 "#PWR0101" H 3650 5950 50  0001 C CNN
-F 1 "VCC" H 3667 6273 50  0000 C CNN
-F 2 "" H 3650 6100 50  0001 C CNN
-F 3 "" H 3650 6100 50  0001 C CNN
-	1    3650 6100
+P 3100 6100
+F 0 "#PWR0101" H 3100 5950 50  0001 C CNN
+F 1 "VCC" H 3117 6273 50  0000 C CNN
+F 2 "" H 3100 6100 50  0001 C CNN
+F 3 "" H 3100 6100 50  0001 C CNN
+	1    3100 6100
 	1    0    0    -1
 $EndComp
@@
 $EndComp
 $Comp
-L power:GND #PWR0104
-U 1 1 5B9B6675
-P 2450 6750
-F 0 "#PWR0104" H 2450 6500 50  0001 C CNN
-F 1 "GND" H 2455 6577 50  0000 C CNN
-F 2 "" H 2450 6750 50  0001 C CNN
-F 3 "" H 2450 6750 50  0001 C CNN
-	1    2450 6750
-	1    0    0    -1
-$EndComp
-$Comp
 L power:GND #PWR0105
 U 1 1 5B9B66AE
-P 3200 6750
-F 0 "#PWR0105" H 3200 6500 50  0001 C CNN
-F 1 "GND" H 3205 6577 50  0000 C CNN
-F 2 "" H 3200 6750 50  0001 C CNN
-F 3 "" H 3200 6750 50  0001 C CNN
-	1    3200 6750
+P 2650 6750
+F 0 "#PWR0105" H 2650 6500 50  0001 C CNN
+F 1 "GND" H 2655 6577 50  0000 C CNN
+F 2 "" H 2650 6750 50  0001 C CNN
+F 3 "" H 2650 6750 50  0001 C CNN
+	1    2650 6750
 	1    0    0    -1
 $EndComp
@@
 L Device:CP C5
 U 1 1 5B9B66E7
-P 3650 6500
-F 0 "C5" H 3768 6546 50  0000 L CNN
-F 1 "CP" H 3768 6455 50  0000 L CNN
-F 2 "Capacitor_SMD:C_0805_2012Metric_Pad1.15x1.40mm_HandSolder" H 3688 6350 50  0001 C CNN
-F 3 "~" H 3650 6500 50  0001 C CNN
-	1    3650 6500
+P 3100 6500
+F 0 "C5" H 3218 6546 50  0000 L CNN
+F 1 "47u/6.3V" H 3100 6400 50  0000 L CNN
+F 2 "Capacitor_SMD:C_0805_2012Metric_Pad1.15x1.40mm_HandSolder" H 3138 6350 50  0001 C CNN
+F 3 "~" H 3100 6500 50  0001 C CNN
+	1    3100 6500
 	1    0    0    -1
 $EndComp
@@
 L power:GND #PWR0106
 U 1 1 5B9B6739
-P 3650 6750
-F 0 "#PWR0106" H 3650 6500 50  0001 C CNN
-F 1 "GND" H 3655 6577 50  0000 C CNN
-F 2 "" H 3650 6750 50  0001 C CNN
-F 3 "" H 3650 6750 50  0001 C CNN
-	1    3650 6750
+P 3100 6750
+F 0 "#PWR0106" H 3100 6500 50  0001 C CNN
+F 1 "GND" H 3105 6577 50  0000 C CNN
+F 2 "" H 3100 6750 50  0001 C CNN
+F 3 "" H 3100 6750 50  0001 C CNN
+	1    3100 6750
 	1    0    0    -1
 $EndComp
@@
 	1300 6250 1300 6350
 Wire Wire Line
-	2250 6250 2450 6250
-Wire Wire Line
-	2450 6250 2450 6350
-Wire Wire Line
-	2450 6650 2450 6750
-Wire Wire Line
-	3200 6650 3200 6750
-Wire Wire Line
-	3650 6650 3650 6750
-Wire Wire Line
-	2450 6250 3200 6250
-Wire Wire Line
-	3200 6250 3200 6350
-Connection ~ 2450 6250
-Wire Wire Line
-	3200 6250 3650 6250
-Wire Wire Line
-	3650 6250 3650 6350
-Connection ~ 3200 6250
-Wire Wire Line
-	3650 6100 3650 6250
-Connection ~ 3650 6250
+	2650 6650 2650 6750
+Wire Wire Line
+	3100 6650 3100 6750
+Wire Wire Line
+	2650 6250 2650 6350
+Wire Wire Line
+	2650 6250 3100 6250
+Wire Wire Line
+	3100 6250 3100 6350
+Connection ~ 2650 6250
+Wire Wire Line
+	3100 6100 3100 6250
+Connection ~ 3100 6250
 $Comp
 L power:GND #PWR0115
@@
 Text Notes 1750 4950 0    50   ~ 0
 The following MCU pins can not be moved:\nCH3-Rx PIO0: ISP UART Rx (you can assign another RC channel though!)\nCH4-Tx PIO4: ISP UART Tx (you can assign another RC channel though!)\nBIND-ISP PIO12: ISP entry button\nXTALIN PIO8: crystal\nXTALIN PIO9: crystal
+$Comp
+L nrf24l01_E01-ML01:NRF24L01_E01_ML01 U3
+U 1 1 5B9F4EE8
+P 6550 2000
+F 0 "U3" H 7027 1978 50  0000 L CNN
+F 1 "NRF24L01_E01_ML01" H 7027 1887 50  0000 L CNN
+F 2 "nordic-semiconductor:nrf24l01-E01-ML01IPX" H 6700 2600 50  0001 L CIN
+F 3 "http://www.nordicsemi.com/eng/content/download/2730/34105/file/nRF24L01_Product_Specification_v2_0.pdf" H 6550 1900 50  0001 C CNN
+	1    6550 2000
+	1    0    0    -1
+$EndComp
+Wire Wire Line
+	2250 6250 2650 6250
 $EndSCHEMATC

Commit message: Tweak layout
Parts:
- removed Y1: 16MHz, Crystal:Crystal_SMD_3225-4Pin_3.2x2.5mm_HandSoldering, symbol Device:Crystal
- added Y1: 12 MHz, Crystal:Crystal_SMD_3225-4Pin_3.2x2.5mm_HandSoldering, symbol Device:Crystal_GND24
Connections:
- no-connect marks 0 -> 2
Changed lines of the file:
@@
-$EndComp
-$Comp
-L Device:Crystal Y1
-U 1 1 5B9B560C
-P 5600 6250
-F 0 "Y1" H 5600 6518 50  0000 C CNN
-F 1 "16MHz" H 5600 6427 50  0000 C CNN
-F 2 "Crystal:Crystal_SMD_3225-4Pin_3.2x2.5mm_HandSoldering" H 5600 6250 50  0001 C CNN
-F 3 "~" H 5600 6250 50  0001 C CNN
-	1    5600 6250
-	-1   0    0    -1
 $EndComp
 $Comp
@@
 Wire Wire Line
 	2250 6250 2650 6250
+$Comp
+L Device:Crystal_GND24 Y1
+U 1 1 5BA0EE7A
+P 5600 6250
+F 0 "Y1" H 5700 6450 50  0000 L CNN
+F 1 "12 MHz" H 5700 6050 50  0000 L CNN
+F 2 "Crystal:Crystal_SMD_3225-4Pin_3.2x2.5mm_HandSoldering" H 5600 6250 50  0001 C CNN
+F 3 "~" H 5600 6250 50  0001 C CNN
+	1    5600 6250
+	1    0    0    -1
+$EndComp
+NoConn ~ 5600 6450
+NoConn ~ 5600 6050
 $EndSCHEMATC

Commit message: Reposition the components
Parts:
- SW1: footprint Button_Switch_SMD:SW_SPST_FSMSM -> tact-switch:Tact switch 6x4x3
Connections:
- net labels added: CH1, CH2-Rx, CH5-Tx, CH6
- net labels removed: CH1-Rx, CH2, CH5, CH6-Tx
Changed lines of the file:
@@
 F 0 "SW1" V 7604 5448 50  0000 L CNN
 F 1 "BIND/ISP" V 7695 5448 50  0000 L CNN
-F 2 "Button_Switch_SMD:SW_SPST_FSMSM" H 7650 5500 50  0001 C CNN
+F 2 "tact-switch:Tact switch 6x4x3" H 7650 5500 50  0001 C CNN
 F 3 "" H 7650 5500 50  0001 C CNN
 	1    7650 5300
@@
 	2500 2700 1900 2700
 Text Label 1900 2700 0    50   ~ 0
-CH1-Rx
+CH2-Rx
 Wire Wire Line
 	2500 2800 1900 2800
@@
 	2500 3400 1900 3400
 Text Label 1900 2800 0    50   ~ 0
-CH5
+CH6
 Text Label 1900 2900 0    50   ~ 0
 MOSI
@@
 MISO
 Text Label 1900 3100 0    50   ~ 0
-CH6-Tx
+CH5-Tx
 Text Label 1900 3200 0    50   ~ 0
 IRQ
@@
 	8050 3800 8800 3800
 Text Label 8050 1500 0    50   ~ 0
-CH1-Rx
+CH1
 Text Label 8050 1600 0    50   ~ 0
-CH2
+CH2-Rx
 Text Label 8050 1700 0    50   ~ 0
 CH3
@@
 CH4
 Text Label 8050 3500 0    50   ~ 0
-CH5
+CH5-Tx
 Text Label 8050 3600 0    50   ~ 0
-CH6-Tx
+CH6
 Text Label 8050 3700 0    50   ~ 0
 CH7
@@
 	3900 3500 4600 3500
 Text Label 4600 3200 2    50   ~ 0
-CH2
+CH1
 $Comp
 L power:PWR_FLAG #FLG0102

Commit message: Changel to 2520 crystal to shrink board to 21x21 mm
Parts:
- Y1: footprint Crystal:Crystal_SMD_3225-4Pin_3.2x2.5mm_HandSoldering -> Crystal:Crystal_SMD_2520-4Pin_2.5x2.0mm
Changed lines of the file:
@@
 F 0 "Y1" H 5700 6450 50  0000 L CNN
 F 1 "12 MHz" H 5700 6050 50  0000 L CNN
-F 2 "Crystal:Crystal_SMD_3225-4Pin_3.2x2.5mm_HandSoldering" H 5600 6250 50  0001 C CNN
+F 2 "Crystal:Crystal_SMD_2520-4Pin_2.5x2.0mm" H 5600 6250 50  0001 C CNN
 F 3 "~" H 5600 6250 50  0001 C CNN
 	1    5600 6250
