File: lpc812-nrf24l01-8ch-receiver/electronics/lpc812-nrf24l01-8ch-receiver.kicad_pcb (KiCad board)
At the start: 2 copper layers, 21 x 21 mm, 23 parts, among them J1 CH1, J2 CH2, J3 CH3/Rx, J4 CH4/Tx, J5 CH5, J6 CH6, J7 CH7, J8 CH8, SW1 BIND/ISP, U1 MCP1703A-3302_SOT23, U2 LPC812M101JDH20, U3 NRF24L01_E01_ML01, Y1 12 MHz

Commit message: More tweaks
Parts:
- moved U1 0.15 mm to (136.9, 82.7)
Routing:
- net VDD: track 15.8 -> 22.9 mm
- net VCC: track 3.73 -> 8.55 mm
